Commit message: URDF Fortschritt

File: Lotti_URDF/Lotti.urdf (robot description, URDF)
Before this commit: robot Lotti, 6 links, 5 joints
Links:
- removed link world
- added link arm_gripper_link, mass 0.2; collision box size=0.08 0.1 0.04; visual box size=0.02 0.08 0.04
- added link arm_link1_link, mass 0.2; collision box size=0.08 0.04 0.1; visual box size=0.08 0.04 0.1
- added link arm_link2_link, mass 0.2; collision box size=0.08 0.04 0.286; visual box size=0.08 0.04 0.286
- added link arm_link3_link, mass 0.2; collision box size=0.08 0.04 0.25; visual box size=0.08 0.04 0.25
- added link arm_link4_link, mass 0.2; collision box size=0.04 0.08 0.1; visual box size=0.04 0.08 0.1
- added link arm_link5_link, mass 0.2; collision box size=0.04 0.04 0.05; visual box size=0.04 0.04 0.05
- link body_link: geometry collision box size=0.7 0.4 0.3; visual box size=0.7 0.4 0.3
Joints:
- removed joint body_joint
- added joint arm_gripper_joint: type fixed, parent arm_link5_link, child arm_gripper_link, origin xyz=0 0 0.05 rpy=0 -1.5707963267948966 0
- added joint arm_link1_joint: type revolute, parent body_link, child arm_link1_link, origin xyz=0.14999999999999997 0.02 0.3 rpy=0 0 0, axis 0 0 1, limit lower=-1.5707963267948966 upper=1.5707963267948966 effort=100 velocity=10
- added joint arm_link2_joint: type revolute, parent arm_link1_link, child arm_link2_link, origin xyz=0 -0.04 0.1 rpy=0 0 0, axis 0 1 0, limit lower=-1.5707963267948966 upper=1.5707963267948966 effort=100 velocity=10
- added joint arm_link3_joint: type revolute, parent arm_link2_link, child arm_link3_link, origin xyz=0 0.04 0.286 rpy=0 0 0, axis 0 1 0, limit lower=-1.5707963267948966 upper=1.5707963267948966 effort=100 velocity=10
- added joint arm_link4_joint: type revolute, parent arm_link3_link, child arm_link4_link, origin xyz=-0.04 -0.02 0.25 rpy=0 0 0, axis 1 0 0, limit lower=-1.0471975511965976 upper=1.0471975511965976 effort=100 velocity=10
- added joint arm_link5_joint: type revolute, parent arm_link4_link, child arm_link5_link, origin xyz=-0.02 0 0.1 rpy=0 0 0, axis 0 0 1, limit lower=-3.141592653589793 upper=3.141592653589793 effort=100 velocity=10
- joint flipper_fl_joint: axis 0 -1 0 -> 0 1 0; limit lower=-1.5707963267948966 upper=1.5707963267948966 effort=100 velocity=10 -> (none); origin xyz=0.19999999999999998 -0.225 0.1 rpy=0 0 0 -> xyz=0.24999999999999997 -0.225 0.1 rpy=0 3.141592653589793 0; type revolute -> continuous
- joint flipper_fr_joint: axis 0 -1 0 -> 0 1 0; limit lower=-1.5707963267948966 upper=1.5707963267948966 effort=100 velocity=10 -> (none); origin xyz=0.19999999999999998 0.225 0.1 rpy=0 0 0 -> xyz=0.24999999999999997 0.225 0.1 rpy=0 3.141592653589793 0; type revolute -> continuous
- joint flipper_rl_joint: limit lower=-1.5707963267948966 upper=1.5707963267948966 effort=100 velocity=10 -> (none); origin xyz=-0.19999999999999998 -0.225 0.1 rpy=0 0 0 -> xyz=-0.24999999999999997 -0.225 0.1 rpy=0 0 0; type revolute -> continuous
- joint flipper_rr_joint: limit lower=-1.5707963267948966 upper=1.5707963267948966 effort=100 velocity=10 -> (none); origin xyz=-0.19999999999999998 0.225 0.1 rpy=0 0 0 -> xyz=-0.24999999999999997 0.225 0.1 rpy=0 0 0; type revolute -> continuous

File: Lotti_URDF/Lotti_main.urdf.xacro (robot description, xacro)
@@ -6,7 +6,10 @@
     <xacro:include filename="Lotti_arm.xacro"/>
     <xacro:include filename="Lotti_body.xacro"/>
+<!--
     <xacro:include filename="Lotti_gazebo_control.xacro"/>
     <xacro:include filename="Lotti_ros2_control.xacro"/>
-<!-- world origin -->
+-->
+<!-- world origin
     <link name="world"></link>
+-->
 </robot>

File: Lotti_URDF/urdf_materials.xacro (robot description, xacro)
@@ -7,3 +7,6 @@
         <color rgba ="${39/255} ${41/255} ${43/255} 1" />
     </material>
+    <material name="orange">
+        <color rgba ="${255/255} ${165/255} ${0/255} 1" />
+    </material>
 </robot>

Commit message: forward urdf

File: Lotti_URDF/Lotti.urdf (robot description, URDF)
Before this commit: robot Lotti, 11 links, 10 joints
Links:
- added link arm_link6_link, mass 0.2; collision box size=0.04 0.04 0.05; visual box size=0.04 0.04 0.05
- link arm_link4_link: geometry collision box size=0.08 0.04 0.1; visual box size=0.08 0.04 0.1
- link arm_link5_link: geometry collision box size=0.04 0.08 0.1; visual box size=0.04 0.08 0.1
Joints:
- added joint arm_link6_joint: type revolute, parent arm_link5_link, child arm_link6_link, origin xyz=-0.02 0 0.1 rpy=0 0 0, axis 0 0 -1, limit lower=-3.141592653589793 upper=3.141592653589793 effort=100 velocity=10
- joint arm_gripper_joint: parent arm_link5_link -> arm_link6_link
- joint arm_link4_joint: axis 1 0 0 -> 0 1 0; limit lower=-1.0471975511965976 upper=1.0471975511965976 effort=100 velocity=10 -> lower=-1.5707963267948966 upper=1.5707963267948966 effort=100 velocity=10; origin xyz=-0.04 -0.02 0.25 rpy=0 0 0 -> xyz=0 0.04 0.25 rpy=0 0 0
- joint arm_link5_joint: axis 0 0 1 -> 1 0 0; limit lower=-3.141592653589793 upper=3.141592653589793 effort=100 velocity=10 -> lower=-1.0471975511965976 upper=1.0471975511965976 effort=100 velocity=10; origin xyz=-0.02 0 0.1 rpy=0 0 0 -> xyz=-0.04 -0.02 0.1 rpy=0 0 0

File: Lotti_URDF/Lotti_arm.xacro (robot description, xacro)
@@ -91,56 +91,83 @@
         </xacro:inertial_box>
     </link>
-<!-- Wrist swivel-->
+<!-- Wrist tilt -->
     <xacro:property name="link4_height" value="0.10"/>
     <joint name="arm_link4_joint" type="revolute">
-        <origin xyz="${-(link_length/2)} ${-link_width/2} ${link3_height}" rpy="0 0 0"/>
+        <origin xyz="0 ${link_width} ${link3_height}" rpy="0 0 0"/>
         <parent link="arm_link3_link"/>
         <child link="arm_link4_link"/>
+        <axis xyz="0 1 0"/>
+        <limit lower="${-pi/2}" upper="${pi/2}" velocity="10" effort="100"/>
+    </joint>
+    <link name="arm_link4_link">
+        <visual>
+            <origin  xyz="0 0 ${link4_height/2}" rpy="0 0 0"/>
+            <geometry>
+                <box size="${link_length} ${link_width} ${link4_height}"/>
+            </geometry>
+            <material name="orange"/>
+        </visual>
+        <collision>
+            <origin  xyz="0 0 ${link4_height/2}" rpy="0 0 0"/>
+            <geometry>
+                <box size="${link_length} ${link_width} ${link4_height}"/>
+            </geometry>
+        </collision>
+        <xacro:inertial_box mass="${link_mass}" x="${link_length}" y="${link_width}" z="${link4_height}">
+            <origin  xyz="0 0 ${link4_height/2}" rpy="0 0 0"/>
+        </xacro:inertial_box>
+    </link>
+<!-- Wrist swivel-->
+    <xacro:property name="link5_height" value="0.10"/>
+    <joint name="arm_link5_joint" type="revolute">
+        <origin xyz="${-(link_length/2)} ${-link_width/2} ${link4_height}" rpy="0 0 0"/>
+        <parent link="arm_link4_link"/>
+        <child link="arm_link5_link"/>
         <axis xyz="1 0 0"/>
         <limit lower="${-pi/3}" upper="${pi/3}" velocity="10" effort="100"/>
     </joint>
-    <link name="arm_link4_link">
-        <visual>
-            <origin  xyz="${-link_width/2} 0 ${link4_height/2}" rpy="0 0 0"/>
-            <geometry>
-                <box size="${link_width} ${link_length} ${link4_height}"/>
-            </geometry>
-            <material name="orange"/>
-        </visual>
-        <collision>
-            <origin  xyz="${-link_width/2} 0 ${link4_height/2}" rpy="0 0 0"/>
-            <geometry>
-                <box size="${link_width} ${link_length} ${link4_height}"/>
-            </geometry>
-        </collision>
-        <xacro:inertial_box mass="${link_mass}" x="${link_width}" y="${link_length}" z="${link4_height}">
-            <origin  xyz="${-link_width/2} 0 ${link4_height/2}" rpy="0 0 0"/>
+    <link name="arm_link5_link">
+        <visual>
+            <origin  xyz="${-link_width/2} 0 ${link5_height/2}" rpy="0 0 0"/>
+            <geometry>
+                <box size="${link_width} ${link_length} ${link5_height}"/>
+            </geometry>
+            <material name="orange"/>
+        </visual>
+        <collision>
+            <origin  xyz="${-link_width/2} 0 ${link5_height/2}" rpy="0 0 0"/>
+            <geometry>
+                <box size="${link_width} ${link_length} ${link5_height}"/>
+            </geometry>
+        </collision>
+        <xacro:inertial_box mass="${link_mass}" x="${link_width}" y="${link_length}" z="${link5_height}">
+            <origin  xyz="${-link_width/2} 0 ${link5_height/2}" rpy="0 0 0"/>
         </xacro:inertial_box>
     </link>
 <!-- Wrist rotate -->
-    <xacro:property name="link5_height" value="0.05"/>
-    <joint name="arm_link5_joint" type="revolute">
-        <origin xyz="${-link_width/2} 0 ${link4_height}" rpy="0 0 0"/>
-        <parent link="arm_link4_link"/>
-        <child link="arm_link5_link"/>
-        <axis xyz="0 0 1"/>
+    <xacro:property name="link6_height" value="0.05"/>
+    <joint name="arm_link6_joint" type="revolute">
+        <origin xyz="${-link_width/2} 0 ${link5_height}" rpy="0 0 0"/>
+        <parent link="arm_link5_link"/>
+        <child link="arm_link6_link"/>
+        <axis xyz="0 0 -1"/>
         <limit lower="${-pi}" upper="${pi}" velocity="10" effort="100"/>
     </joint>
-    <link name="arm_link5_link">
-        <visual>
-            <origin  xyz="0 0 ${link5_height/2}" rpy="0 0 0"/>
-            <geometry>
-                <box size="${link_width} ${link_width} ${link5_height}"/>
-            </geometry>
-            <material name="orange"/>
-        </visual>
-        <collision>
-            <origin  xyz="0 0 ${link5_height/2}" rpy="0 0 0"/>
-            <geometry>
-                <box size="${link_width} ${link_width} ${link5_height}"/>
-            </geometry>
-        </collision>
-        <xacro:inertial_box mass="${link_mass}" x="${link_width}" y="${link_width}" z="${link5_height}">
-            <origin  xyz="0 0 ${link5_height/2}" rpy="0 0 0"/>
+    <link name="arm_link6_link">
+        <visual>
+            <origin  xyz="0 0 ${link6_height/2}" rpy="0 0 0"/>
+            <geometry>
+                <box size="${link_width} ${link_width} ${link6_height}"/>
+            </geometry>
+            <material name="orange"/>
+        </visual>
+        <collision>
+            <origin  xyz="0 0 ${link6_height/2}" rpy="0 0 0"/>
+            <geometry>
+                <box size="${link_width} ${link_width} ${link6_height}"/>
+            </geometry>
+        </collision>
+        <xacro:inertial_box mass="${link_mass}" x="${link_width}" y="${link_width}" z="${link6_height}">
+            <origin  xyz="0 0 ${link6_height/2}" rpy="0 0 0"/>
         </xacro:inertial_box>
     </link>
@@ -150,6 +177,6 @@
     <xacro:property name="gripper_length" value="0.08"/>
     <joint name="arm_gripper_joint" type="fixed">
-        <origin xyz="0 0 ${link5_height}" rpy="0 ${-pi/2} 0"/>
-        <parent link="arm_link5_link"/>
+        <origin xyz="0 0 ${link6_height}" rpy="0 ${-pi/2} 0"/>
+        <parent link="arm_link6_link"/>
         <child link="arm_gripper_link"/>
     </joint>

File: Lotti_URDF/Lotti_ros_control.xacro (robot description, xacro)
@@ -1,5 +1,6 @@
 <?xml version="1.0"?>
 <robot xmlns:xacro="http://www.ros.org/wiki/xacro" >
-    <ros2_control name="LottiControlls" type="system">
+<!-- left chain -->
+    <ros2_control name="left_chain_control" type="actuator">
         <hardware>
             <plugin>gazebo_ros2_control/LottiControlls</plugin>
@@ -14,3 +15,31 @@
         </joint>
     </ros2_control>
+<!-- right chain -->
+    <ros2_control name="right_chain_control" type="actuator">
+        <hardware>
+            <plugin>ros2_control_demo_hardware/PositionActuatorHardware</plugin>
+            <param name="example_param_write_for_sec">1.23</param>
+            <param name="example_param_read_for_sec">3</param>
+        </hardware>
+        <joint name="joint1">
+            <command_interface name="position">
+                <param name="min">-1</param>
+                <param name="max">1</param>
+            </command_interface>
+            <state_interface name="position"/>
+        </joint>
+    </ros2_control>
+<!-- front right flipper -->
+    <ros2_control name="flipper_fr_control" type="actuator">
+        <hardware>
+        </hardware>
+        <joint name="flipper_fr_joint">
+            <command_interface name="velocity">
+                <param name="min">-1</param>
+                <param name="max">1</param>
+                <param name="initial_value">0</param>
+            </command_interface>
+            <state_interface name="position"/>
+        </joint>
+    </ros2_control>
 </robot>
