Commit message: arm controlls working

File: control_ws/src/lotti_control/description/srdf/lotti_body_group.xacro (robot description, xacro)
@@ -7,17 +7,28 @@
     <!--CHAINS: When a chain is specified, all the links along the chain (including endpoints) are included in the group. Additionally, all the joints that are parents to included links are also included. This means that joints along the chain and the parent joint of the base link are included in the group-->
     <!--SUBGROUPS: Groups can also be formed by referencing to already defined group names-->
-    <group name="hand">
-      <link name="panda_hand" />
-      <link name="panda_leftfinger" />
-      <link name="panda_rightfinger" />
-      <joint name="panda_finger_joint1" />
-      <passive_joint name="panda_finger_joint2" />
+    <group name="lotti_body">
+      <link name="body_link" />
+      <link name="flipper_fr_link" />
+      <link name="flipper_rr_link" />
+      <joint name="flipper_fl_link" />
+      <joint name="flipper_rl_link" />
+      <joint name="right_main_wheel_link" />
+      <joint name="left_main_wheel_link" />
     </group>
     <!--GROUP STATES: Purpose: Define a named state for a particular group, in terms of joint values. This is useful to define states like 'folded arms'-->
     <!--END EFFECTOR: Purpose: Represent information about an end effector.-->
     <!--DISABLE COLLISIONS: By default it is assumed that any link of the robot could potentially come into collision with any other link in the robot. This tag disables collision checking between a specified pair of links. -->
-    <disable_collisions link1="panda_hand" link2="panda_leftfinger" reason="Adjacent" />
-    <disable_collisions link1="panda_hand" link2="panda_rightfinger" reason="Adjacent" />
-    <disable_collisions link1="panda_leftfinger" link2="panda_rightfinger" reason="Default" />
+      <!-- body_link never collides with rest of body parts -->
+    <disable_collisions link1="body_link" link2="left_main_wheel_link" reason="Never" />
+    <disable_collisions link1="body_link" link2="right_main_wheel_link" reason="Never" />
+    <disable_collisions link1="body_link" link2="flipper_fr_link" reason="Never" />
+    <disable_collisions link1="body_link" link2="flipper_fl_link" reason="Never" />
+    <disable_collisions link1="body_link" link2="flipper_rr_link" reason="Never" />
+    <disable_collisions link1="body_link" link2="flipper_rl_link" reason="Never" />
+      <!-- right flippers never collide with left flippers -->
+    <disable_collisions link1="flipper_fl_link" link2="flipper_rr_link" reason="Never" />
+    <disable_collisions link1="flipper_rl_link" link2="flipper_rr_link" reason="Never" />
+    <disable_collisions link1="flipper_fl_link" link2="flipper_fr_link" reason="Never" />
+    <disable_collisions link1="flipper_rl_link" link2="flipper_fr_link" reason="Never" />
   </xacro:macro>
 </robot>

File: old stuff/lotti_moveit_control/config/Lotti_arm.xacro (robot description, xacro)
@@ -30,5 +30,5 @@
             <origin  xyz="0 0 ${link1_height/2}" rpy="0 0 0"/>
             <geometry>
-                <box size="${link_length -0.021} ${link_width -0.021} ${link1_height -0.021}"/>
+                <box size="${link_length} ${link_width} ${link1_height}"/>
             </geometry>
         </collision>
@@ -40,9 +40,9 @@
     <xacro:property name="link2_height" value="0.286"/>
     <joint name="arm_link2_joint" type="revolute">
-        <origin xyz="0 ${-link_width} ${link1_height}" rpy="0 -1.1 0"/>
+        <origin xyz="0 ${-link_width} ${link1_height}" rpy="0 0 0"/>
         <parent link="arm_link1_link"/>
         <child link="arm_link2_link"/>
         <axis xyz="0 1 0"/>
-        <limit lower="-0.2" upper="2.8" velocity="10" effort="100"/>
+        <limit lower="-1.2" upper="1.2" velocity="10" effort="100"/>
     </joint>
     <link name="arm_link2_link">
@@ -57,5 +57,5 @@
             <origin  xyz="0 0 ${link2_height/2}" rpy="0 0 0"/>
             <geometry>
-                <box size="${link_length -0.021} ${link_width -0.021} ${link2_height -0.021}"/>
+                <box size="${link_length} ${link_width} ${link2_height}"/>
             </geometry>
         </collision>
@@ -67,9 +67,9 @@
     <xacro:property name="link3_height" value="0.25"/>
     <joint name="arm_link3_joint" type="revolute">
-        <origin xyz="0 ${link_width} ${link2_height}" rpy="0 2.4 0"/>
+        <origin xyz="0 ${link_width} ${link2_height}" rpy="0 0 0"/>
         <parent link="arm_link2_link"/>
         <child link="arm_link3_link"/>
         <axis xyz="0 1 0"/>
-        <limit lower="-2.2" upper="0.4" velocity="10" effort="100"/>
+        <limit lower="${-pi}" upper="${pi}" velocity="10" effort="100"/>
     </joint>
     <link name="arm_link3_link">
@@ -84,5 +84,5 @@
             <origin  xyz="0 0 ${link3_height/2}" rpy="0 0 0"/>
             <geometry>
-                <box size="${link_length -0.021} ${link_width -0.021} ${link3_height -0.021}"/>
+                <box size="${link_length} ${link_width} ${link3_height}"/>
             </geometry>
         </collision>
@@ -94,5 +94,5 @@
     <xacro:property name="link4_height" value="0.10"/>
     <joint name="arm_link4_joint" type="revolute">
-        <origin xyz="0 ${link_width} ${link3_height}" rpy="0 ${(pi/2) -1.3} 0"/>
+        <origin xyz="0 ${link_width} ${link3_height}" rpy="0 0 0"/>
         <parent link="arm_link3_link"/>
         <child link="arm_link4_link"/>
@@ -111,5 +111,5 @@
             <origin  xyz="0 0 ${link4_height/2}" rpy="0 0 0"/>
             <geometry>
-                <box size="${link_length -0.021} ${link_width -0.021} ${link4_height -0.021}"/>
+                <box size="${link_length} ${link_width} ${link4_height}"/>
             </geometry>
         </collision>
@@ -138,5 +138,5 @@
             <origin  xyz="${-link_width/2} 0 ${link5_height/2}" rpy="0 0 0"/>
             <geometry>
-                <box size="${link_width -0.021} ${link_length -0.021} ${link5_height -0.021}"/>
+                <box size="${link_width} ${link_length} ${link5_height}"/>
             </geometry>
         </collision>
@@ -165,5 +165,5 @@
             <origin  xyz="0 0 ${link6_height/2}" rpy="0 0 0"/>
             <geometry>
-                <box size="${link_width -0.021} ${link_width -0.021} ${link6_height -0.021}"/>
+                <box size="${link_width} ${link_width} ${link6_height}"/>
             </geometry>
         </collision>

File: old stuff/lotti_moveit_control/config/Lotti_body.xacro (robot description, xacro)
@@ -6,10 +6,4 @@
     <xacro:property name="body_height" value="0.15"/>
     <xacro:property name="body_mass" value="25.0"/>
-    <joint name="world_joint" type="fixed">
-        <origin xyz="0 0 0" rpy="0 0 0"/>
-        <parent link="world"/>
-        <child link="body_link"/>
-        <axis xyz="0 0 0"/>
-    </joint>
     <link name="body_link">
         <visual>
