Commit message: cool arm working

File: control_ws/src/lotti_control/description/urdf/Lotti_arm.xacro (robot description, xacro)
@@ -1,215 +1,235 @@
-<?xml version="1.0"?>
+<?xml version="1.0" encoding="utf-8"?>
+<!-- This URDF was automatically created by SolidWorks to URDF Exporter! Originally created by Stephen Brawner (brawner@gmail.com)
+     Commit Version: 1.6.0-4-g7f85cfe  Build Version: 1.6.7995.38578
+     For more information, please see http://wiki.ros.org/sw_urdf_exporter -->
 <robot xmlns:xacro="http://www.ros.org/wiki/xacro" >
-<!-- Rotating Base -->
-    <!-- Body params for reference -->
-    <xacro:property name="body_length" value="0.7"/>
-    <xacro:property name="body_width" value="0.33"/>
-    <xacro:property name="body_height" value="0.15"/>
-    <!-- same for all links -->
-    <xacro:property name="link_length" value="0.08"/>
-    <xacro:property name="link_width" value="0.04"/>
-    <xacro:property name="link_mass" value="0.2"/>
-    <!-- changing param -->
-    <xacro:property name="link1_height" value="0.10"/>
-    <joint name="arm_link1_joint" type="revolute">
-        <origin xyz="${body_length/2 - 0.1} ${link_width/2} ${body_height}" rpy="0 0 0"/>
-        <parent link="body_link"/>
-        <child link="arm_link1_link"/>
-        <axis xyz="0 0 1"/>
-        <limit lower="${-pi}" upper="${pi}" velocity="10" effort="100"/>
-    </joint>
-    <link name="arm_link1_link">
-        <visual>
-            <origin  xyz="0 0 ${link1_height/2}" rpy="0 0 0"/>
-            <geometry>
-                <box size="${link_length} ${link_width} ${link1_height}"/>
-            </geometry>
-            <material name="orange"/>
-        </visual>
-        <collision>
-            <origin  xyz="0 0 ${link1_height/2}" rpy="0 0 0"/>
-            <geometry>
-                <box size="${link_length -0.021} ${link_width -0.021} ${link1_height -0.021}"/>
-            </geometry>
-        </collision>
-        <xacro:inertial_box mass="${link_mass}" x="${link_length}" y="${link_width}" z="${link1_height}">
-            <origin  xyz="0 0 ${link1_height/2}" rpy="0 0 0"/>
-        </xacro:inertial_box>
-    </link>
-<!-- Lifting Base -->
-    <xacro:property name="link2_height" value="0.286"/>
-    <joint name="arm_link2_joint" type="revolute">
-        <origin xyz="0 ${-link_width} ${link1_height}" rpy="0 -1.1 0"/>
-        <parent link="arm_link1_link"/>
-        <child link="arm_link2_link"/>
-        <axis xyz="0 1 0"/>
-        <limit lower="-0.2" upper="2.8" velocity="10" effort="100"/>
-    </joint>
-    <link name="arm_link2_link">
-        <visual>
-            <origin  xyz="0 0 ${link2_height/2}" rpy="0 0 0"/>
-            <geometry>
-                <box size="${link_length} ${link_width} ${link2_height}"/>
-            </geometry>
-            <material name="orange"/>
-        </visual>
-        <collision>
-            <origin  xyz="0 0 ${link2_height/2}" rpy="0 0 0"/>
-            <geometry>
-                <box size="${link_length -0.021} ${link_width -0.021} ${link2_height -0.021}"/>
-            </geometry>
-        </collision>
-        <xacro:inertial_box mass="${link_mass}" x="${link_length}" y="${link_width}" z="${link2_height}">
-            <origin  xyz="0 0 ${link2_height/2}" rpy="0 0 0"/>
-        </xacro:inertial_box>
-    </link>
-<!-- Elbow -->
-    <xacro:property name="link3_height" value="0.25"/>
-    <joint name="arm_link3_joint" type="revolute">
-        <origin xyz="0 ${link_width} ${link2_height}" rpy="0 2.4 0"/>
-        <parent link="arm_link2_link"/>
-        <child link="arm_link3_link"/>
-        <axis xyz="0 1 0"/>
-        <limit lower="-2.2" upper="0.4" velocity="10" effort="100"/>
-    </joint>
-    <link name="arm_link3_link">
-        <visual>
-            <origin  xyz="0 0 ${link3_height/2}" rpy="0 0 0"/>
-            <geometry>
-                <box size="${link_length} ${link_width} ${link3_height}"/>
-            </geometry>
-            <material name="orange"/>
-        </visual>
-        <collision>
-            <origin  xyz="0 0 ${link3_height/2}" rpy="0 0 0"/>
-            <geometry>
-                <box size="${link_length -0.021} ${link_width -0.021} ${link3_height -0.021}"/>
-            </geometry>
-        </collision>
-        <xacro:inertial_box mass="${link_mass}" x="${link_length}" y="${link_width}" z="${link3_height}">
-            <origin  xyz="0 0 ${link3_height/2}" rpy="0 0 0"/>
-        </xacro:inertial_box>
-    </link>
-<!-- Wrist tilt -->
-    <xacro:property name="link4_height" value="0.10"/>
-    <joint name="arm_link4_joint" type="revolute">
-        <origin xyz="0 ${link_width} ${link3_height}" rpy="0 ${(pi/2) -1.3} 0"/>
-        <parent link="arm_link3_link"/>
-        <child link="arm_link4_link"/>
-        <axis xyz="0 1 0"/>
-        <limit lower="${-pi/2}" upper="${pi/2}" velocity="10" effort="100"/>
-    </joint>
-    <link name="arm_link4_link">
-        <visual>
-            <origin  xyz="0 0 ${link4_height/2}" rpy="0 0 0"/>
-            <geometry>
-                <box size="${link_length} ${link_width} ${link4_height}"/>
-            </geometry>
-            <material name="orange"/>
-        </visual>
-        <collision>
-            <origin  xyz="0 0 ${link4_height/2}" rpy="0 0 0"/>
-            <geometry>
-                <box size="${link_length -0.021} ${link_width -0.021} ${link4_height -0.021}"/>
-            </geometry>
-        </collision>
-        <xacro:inertial_box mass="${link_mass}" x="${link_length}" y="${link_width}" z="${link4_height}">
-            <origin  xyz="0 0 ${link4_height/2}" rpy="0 0 0"/>
-        </xacro:inertial_box>
-    </link>
-<!-- Wrist swivel-->
-    <xacro:property name="link5_height" value="0.10"/>
-    <joint name="arm_link5_joint" type="revolute">
-        <origin xyz="${-(link_length/2)} ${-link_width/2} ${link4_height}" rpy="0 0 0"/>
-        <parent link="arm_link4_link"/>
-        <child link="arm_link5_link"/>
-        <axis xyz="1 0 0"/>
-        <limit lower="${-pi/3}" upper="${pi/3}" velocity="10" effort="100"/>
-    </joint>
-    <link name="arm_link5_link">
-        <visual>
-            <origin  xyz="${-link_width/2} 0 ${link5_height/2}" rpy="0 0 0"/>
-            <geometry>
-                <box size="${link_width} ${link_length} ${link5_height}"/>
-            </geometry>
-            <material name="orange"/>
-        </visual>
-        <collision>
-            <origin  xyz="${-link_width/2} 0 ${link5_height/2}" rpy="0 0 0"/>
-            <geometry>
-                <box size="${link_width -0.021} ${link_length -0.021} ${link5_height -0.021}"/>
-            </geometry>
-        </collision>
-        <xacro:inertial_box mass="${link_mass}" x="${link_width}" y="${link_length}" z="${link5_height}">
-            <origin  xyz="${-link_width/2} 0 ${link5_height/2}" rpy="0 0 0"/>
-        </xacro:inertial_box>
-    </link>
-<!-- Wrist rotate -->
-    <xacro:property name="link6_height" value="0.05"/>
-    <joint name="arm_link6_joint" type="revolute">
-        <origin xyz="${-link_width/2} 0 ${link5_height}" rpy="0 0 0"/>
-        <parent link="arm_link5_link"/>
-        <child link="arm_link6_link"/>
-        <axis xyz="0 0 -1"/>
-        <limit lower="${-pi}" upper="${pi}" velocity="10" effort="100"/>
-    </joint>
-    <link name="arm_link6_link">
-        <visual>
-            <origin  xyz="0 0 ${link6_height/2}" rpy="0 0 0"/>
-            <geometry>
-                <box size="${link_width} ${link_width} ${link6_height}"/>
-            </geometry>
-            <material name="orange"/>
-        </visual>
-        <collision>
-            <origin  xyz="0 0 ${link6_height/2}" rpy="0 0 0"/>
-            <geometry>
-                <box size="${link_width -0.021} ${link_width -0.021} ${link6_height -0.021}"/>
-            </geometry>
-        </collision>
-        <xacro:inertial_box mass="${link_mass}" x="${link_width}" y="${link_width}" z="${link6_height}">
-            <origin  xyz="0 0 ${link6_height/2}" rpy="0 0 0"/>
-        </xacro:inertial_box>
-    </link>
-<!-- Gripper -->
-    <xacro:property name="gripper_height" value="0.04"/>
-    <xacro:property name="gripper_width" value="0.1"/>
-    <xacro:property name="gripper_length" value="0.08"/>
-    <joint name="arm_gripper_joint" type="fixed">
-        <origin xyz="0 0 ${link6_height}" rpy="0 ${-pi/2} 0"/>
-        <parent link="arm_link6_link"/>
-        <child link="arm_gripper_link"/>
-    </joint>
-    <link name="arm_gripper_link">
-        <visual>
-            <origin  xyz="0.01 0 0" rpy="0 0 0"/>
-            <geometry>
-                <box size="0.02 0.08 0.04"/>
-            </geometry>
-            <material name="black"/>
-        </visual>
-        <visual>
-            <origin xyz="0.05 0.03 0" rpy="0 0 0"/>
-            <geometry>
-                <box size="0.06 0.02 0.04"/>
-            </geometry>
-            <material name="black"/>
-        </visual>
-        <visual>
-            <origin xyz="0.05 -0.03 0" rpy="0 0 0"/>
-            <geometry>
-                <box size="0.06 0.02 0.04"/>
-            </geometry>
-            <material name="black"/>
-        </visual>
-        <collision>
-            <origin  xyz="${gripper_length/2} 0 0" rpy="0 0 0"/>
-            <geometry>
-                <box size="${gripper_length} ${gripper_width} ${gripper_height}"/>
-            </geometry>
-        </collision>
-        <xacro:inertial_box mass="${link_mass}" x="${gripper_length}" y="${gripper_width}" z="${gripper_height}">
-            <origin  xyz="${gripper_length/2} 0 0" rpy="0 0 0"/>
-        </xacro:inertial_box>
-    </link>
+<!-- Main Body info -->
+  <xacro:property name="body_length" value="0.7"/>
+  <xacro:property name="body_width" value="0.33"/>
+  <xacro:property name="body_height" value="0.15"/>
+  <xacro:property name="body_mass" value="25.0"/>
+   <joint name="arm_base_joint" type="fixed">
+    <origin xyz="${body_length/2 - 0.1} 0 ${body_height}" rpy="0 0 ${pi}" />
+    <parent link="body_link" />
+    <child link="arm_base_link" />
+  </joint>
+  <link name="arm_base_link">
+    <inertial>
+      <origin xyz="-0.00263222915365038 -0.000332098550481226 0.0476250352231148" rpy="0 0 0" />
+      <mass value="0.200226640012258" />
+      <inertia ixx="0.00030515518623871" ixy="5.9193755234795E-09" ixz="-5.48255039093506E-06"
+               iyy="0.000183595401496948" iyz="3.03172951946039E-10" izz="0.000356726067861412" />
+    </inertial>
+    <visual>
+      <origin xyz="0 0 0" rpy="0 0 0" />
+      <geometry>
+        <mesh filename="package://lotti_control/description/meshes/arm_base_link.STL" />
+      </geometry>
+      <material name="black"/>
+    </visual>
+    <collision>
+      <origin xyz="0 0 0" rpy="0 0 0" />
+      <geometry>
+        <mesh filename="package://lotti_control/description/meshes/arm_base_link.STL" />
+      </geometry>
+    </collision>
+  </link>
+  <link name="arm_link1_link">
+    <inertial>
+      <origin xyz="4.41542086226931E-09 0.000122631739122248 0.0356096098271416" rpy="0 0 0" />
+      <mass value="0.227235996796303" />
+      <inertia ixx="0.000180809625442164" ixy="1.99972159337586E-12" ixz="3.65735427518995E-13"
+               iyy="0.000141436764733896" iyz="-1.12077733619125E-07" izz="0.000174149091246638" />
+    </inertial>
+    <visual>
+      <origin xyz="0 0 0" rpy="0 0 0" />
+      <geometry>
+        <mesh filename="package://lotti_control/description/meshes/arm_link1_link.STL" />
+      </geometry>
+      <material name="red"/>
+    </visual>
+    <collision>
+      <origin xyz="0 0 0" rpy="0 0 0" />
+      <geometry>
+        <mesh filename="package://lotti_control/description/meshes/arm_link1_link.STL" />
+      </geometry>
+    </collision>
+  </link>
+  <joint name="arm_link1_joint" type="revolute">
+    <origin xyz="0 0 0.0813" rpy="0 0 1.5708" />
+    <parent link="arm_base_link" />
+    <child link="arm_link1_link" />
+    <axis xyz="0 0 -1" />
+    <limit
+      lower="-3"
+      upper="3"
+      effort="3"
+      velocity="2" />
+  </joint>
+  <link name="arm_link2_link">
+    <inertial>
+      <origin xyz="-0.0048507016693122 0.000134479355761746 0.151153269049844" rpy="0 0 0" />
+      <mass value="0.308407355142343" />
+      <inertia ixx="0.000536262443976751" ixy="-5.59401799937812E-07" ixz="4.55969735855309E-05"
+               iyy="0.000463619869555736" iyz="-5.41211706294874E-05" izz="0.00028846239166877" />
+    </inertial>
+    <visual>
+      <origin xyz="0 0 0" rpy="0 0 0" />
+      <geometry>
+        <mesh filename="package://lotti_control/description/meshes/arm_link2_link.STL" />
+      </geometry>
+      <material name="">
+        <color
+          rgba="0.792156862745098 0.819607843137255 0.933333333333333 1" />
+      </material>
+    </visual>
+    <collision>
+      <origin xyz="0 0 0" rpy="0 0 0" />
+      <geometry>
+        <mesh filename="package://lotti_control/description/meshes/arm_link2_link.STL" />
+      </geometry>
+    </collision>
+  </link>
+  <joint name="arm_link2_joint" type="revolute">
+    <origin xyz="0 0.002 0.093" rpy="0 1.4835 -1.5708" />
+    <parent link="arm_link1_link" />
+    <child link="arm_link2_link" />
+    <axis xyz="0 1 0" />
+    <limit
+      lower="-1.5"
+      upper="1.5"
+      effort="3"
+      velocity="2" />
+  </joint>
+  <link name="arm_link3_link">
+    <inertial>
+      <origin xyz="-2.34730375641978E-05 0.000222724116048956 0.121657320094858" rpy="0 0 0" />
+      <mass value="0.215223683624819" />
+      <inertia ixx="0.000187887481718192" ixy="1.29568722040644E-09" ixz="-2.48383575759051E-09"
+               iyy="0.000177005795528886" iyz="-1.95381298527238E-05" izz="5.96362197609908E-05" />
+    </inertial>
+    <visual>
+      <origin xyz="0 0 0" rpy="0 0 0" />
+      <geometry>
+        <mesh filename="package://lotti_control/description/meshes/arm_link3_link.STL" />
+      </geometry>
+      <material name="">
+        <color
+          rgba="0.792156862745098 0.819607843137255 0.933333333333333 1" />
+      </material>
+    </visual>
+    <collision>
+      <origin xyz="0 0 0" rpy="0 0 0" />
+      <geometry>
+        <mesh filename="package://lotti_control/description/meshes/arm_link3_link.STL" />
+      </geometry>
+    </collision>
+  </link>
+  <joint name="arm_link3_joint" type="revolute">
+    <origin xyz="-0.05 0 0.29" rpy="-3.1416 -0.087266 -3.1416" />
+    <parent link="arm_link2_link" />
+    <child link="arm_link3_link" />
+    <axis xyz="0 1 0" />
+    <limit
+      lower="0"
+      upper="2.9"
+      effort="3"
+      velocity="2" />
+  </joint>
+  <link name="arm_link4_link">
+    <inertial>
+      <origin xyz="-6.45090288222683E-05 -2.78077069245236E-05 0.0421410408275518" rpy="0 0 0" />
+      <mass value="0.0799976203193007" />
+      <inertia ixx="2.98275167277768E-05" ixy="-3.7887086534939E-10" ixz="2.42643938146603E-10"
+               iyy="1.60577540866642E-05" iyz="1.06831058124334E-09" izz="2.00421216012606E-05" />
+    </inertial>
+    <visual>
+      <origin xyz="0 0 0" rpy="0 0 0" />
+      <geometry>
+        <mesh filename="package://lotti_control/description/meshes/arm_link4_link.STL" />
+      </geometry>
+      <material name="red"/>
+    </visual>
+    <collision>
+      <origin xyz="0 0 0" rpy="0 0 0" />
+      <geometry>
+        <mesh filename="package://lotti_control/description/meshes/arm_link4_link.STL" />
+      </geometry>
+    </collision>
+  </link>
+  <joint name="arm_link4_joint" type="revolute">
+    <origin xyz="0 0.0006 0.26473" rpy="0 0 0" />
+    <parent link="arm_link3_link" />
+    <child link="arm_link4_link" />
+    <axis xyz="0 1 0" />
+    <limit
+      lower="-1.5"
+      upper="1.5"
+      effort="3"
+      velocity="2" />
+  </joint>
+  <link name="arm_link5_link">
+    <inertial>
+      <origin xyz="0.00382150605784218 -7.85621768924077E-05 0.0340017507140268" rpy="0 0 0" />
+      <mass value="0.0824183861074926" />
+      <inertia ixx="1.34651970301422E-05" ixy="1.06510176549428E-09" ixz="7.33151583060291E-09"
+               iyy="3.06523685609497E-05" iyz="3.77177397775468E-10" izz="3.09091303833254E-05" />
+    </inertial>
+    <visual>
+      <origin xyz="0 0 0" rpy="0 0 0" />
+      <geometry>
+        <mesh filename="package://lotti_control/description/meshes/arm_link5_link.STL" />
+      </geometry>
+      <material name="black"/>
+    </visual>
+    <collision>
+      <origin xyz="0 0 0" rpy="0 0 0" />
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
File: control_ws/src/lotti_control/description/urdf/Lotti_body.xacro (robot description, xacro)
@@ -6,5 +6,5 @@
     <xacro:property name="body_height" value="0.15"/>
     <xacro:property name="body_mass" value="25.0"/>
-<!--     <joint name="world_joint" type="floating">
+    <!-- <joint name="world_joint" type="floating">
         <origin xyz="0 0 0" rpy="0 0 0"/>
         <parent link="world"/>

Commit message: all in one

File: control_ws/src/lotti_control/description/urdf/Lotti_arm.xacro (robot description, xacro)
@@ -159,11 +159,11 @@
   </link>
   <joint name="arm_link4_joint" type="revolute">
-    <origin xyz="0 0.0006 0.26473" rpy="0 0 0" />
+    <origin xyz="0 0.0006 0.26473" rpy="0 -1.5 0" />
     <parent link="arm_link3_link" />
     <child link="arm_link4_link" />
     <axis xyz="0 1 0" />
     <limit
-      lower="-1.5"
-      upper="1.5"
+      lower="0"
+      upper="3"
       effort="3"
       velocity="1" />
@@ -191,11 +191,11 @@
   </link>
   <joint name="arm_link5_joint" type="revolute">
-    <origin xyz="-0.00055 0.0001 0.074331" rpy="0 0 0" />
+    <origin xyz="-0.00055 0.0001 0.074331" rpy="-1.5 0 0" />
     <parent link="arm_link4_link" />
     <child link="arm_link5_link" />
     <axis xyz="1 0 0" />
     <limit
-      lower="-1.5"
-      upper="1.5"
+      lower="0"
+      upper="3"
       effort="3"
       velocity="1" />

File: control_ws/src/lotti_control/description/urdf/Lotti_body.xacro (robot description, xacro)
@@ -32,5 +32,5 @@
         </xacro:inertial_box> -->
     </link>
-<!-- Chains (represented by three wheels each, only the middle one beeing motorized) -->
+<!-- Chains (represented by wheels) -->
 <!-- wheel macro-->
     <xacro:property name="wheel_length" value="0.15"/>
@@ -67,19 +67,4 @@
     </joint>
     <xacro:wheel_link position="left_main"/>
-<!-- Support Wheels-->
-<!--     <joint name="left_chain_support1_joint" type="continuous">
-        <origin xyz="${(body_length/2) - wheel_radius} ${wheel_seperation/2} ${wheel_radius}" rpy="0 0 0"/>
-        <parent link="body_link"/>
-        <child link="left_support1_wheel_link"/>
-        <axis xyz="0 1 0"/>
-    </joint>
-    <xacro:wheel_link position="left_support1"/>
-    <joint name="left_chain_support2_joint" type="continuous">
-        <origin xyz="${-(body_length/2) + wheel_radius} ${wheel_seperation/2} ${wheel_radius}" rpy="0 0 0"/>
-        <parent link="body_link"/>
-        <child link="left_support2_wheel_link"/>
-        <axis xyz="0 1 0"/>
-    </joint>
-    <xacro:wheel_link position="left_support2"/> -->
 <!-- Right Chain-->
 <!-- Main Wheel-->
@@ -91,25 +76,9 @@
     </joint>
     <xacro:wheel_link position="right_main"/>
-<!-- Support Wheels-->
-<!--     <joint name="right_chain_support1_joint" type="continuous">
-        <origin xyz="${(body_length/2) - wheel_radius} ${-wheel_seperation/2} ${wheel_radius}" rpy="0 0 0"/>
-        <parent link="body_link"/>
-        <child link="right_support1_wheel_link"/>
-        <axis xyz="0 -1 0"/>
-    </joint>
-    <xacro:wheel_link position="right_support1"/>
-    <joint name="right_chain_support2_joint" type="continuous">
-        <origin xyz="${-(body_length/2) + wheel_radius} ${-wheel_seperation/2} ${wheel_radius}" rpy="0 0 0"/>
-        <parent link="body_link"/>
-        <child link="right_support2_wheel_link"/>
-        <axis xyz="0 -1 0"/>
-    </joint>
-    <xacro:wheel_link position="right_support2"/>
- -->
 <!-- Flipper -->
     <xacro:property name="flipper_length" value="0.4"/>
     <xacro:property name="flipper_width" value="0.05"/>
     <xacro:property name="flipper_height" value="0.2"/>
-    <xacro:property name="flipper_mass" value="3.0"/>
+    <xacro:property name="flipper_mass" value="2.0"/>
 <!-- Flipper link macro -->
     <xacro:macro name="flipper_link" params="position">
@@ -173,3 +142,26 @@
     </joint>
     <xacro:flipper_link position="rl"/>
+<!-- Sensors -->
+    <!-- LiDAR -->
+    <joint name="lidar_joint" type="fixed">
+        <origin xyz="-0.3 0 0.25" rpy="0 ${-30*pi/180} 0"/>
+        <parent link="body_link"/>
+        <child link="lidar_link"/>
+    </joint>
+    <link name="lidar_link">
+        <visual>
+            <origin rpy="0 0 0" xyz="0 0 0"/>
+            <geometry>
+                <box size="0.06 0.06 0.06"/>
+            </geometry>
+            <material name="orange"/>
+        </visual>
+        <collision>
+            <origin rpy="0 0 0" xyz="0 0 0"/>
+            <geometry>
+                <box size="0.06 0.06 0.06"/>
+            </geometry>
+        </collision>
+        <innertial></innertial>
+    </link>
 </robot>
