Commit message: Add Livox Mid-360 + Nav2 autonomous navigation stack
- Fix lidar_link position (30cm fwd, 30cm left, 30deg pitch back)
- Add Livox ROS2 driver + pointcloud_to_laserscan to robot.launch.py
- Add MID360_config.json (set sensor IP before use)
- Add nav2_params.yaml with PointCloud2 + LaserScan dual obstacle sources
- Add slam_toolbox_params.yaml for online async SLAM
- Wire slam_toolbox + Nav2 + cmd_vel relay into operator.launch.py
- Update RViz: add Map, Costmaps, LaserScan, PointCloud2, Path displays
- Change RViz Fixed Frame to map

Co-Authored-By: Claude Sonnet 4.6 <noreply@anthropic.com>

File: control_ws/src/lotti_control/description/urdf/Lotti_lidar.xacro (robot description, xacro)
@@ -2,5 +2,7 @@
 <robot xmlns:xacro="http://www.ros.org/wiki/xacro" >
     <joint name="lidar_joint" type="fixed">
-        <origin xyz="0 0 0" rpy="0 0 0"/>
+        <!-- 30cm forward, 30cm left of robot origin, 0cm vertical -->
+        <!-- pitch = +0.5236 rad (30°): sensor top tilts toward rear -->
+        <origin xyz="0.30 0.30 0.0" rpy="0 0.5236 0"/>
         <parent link="body_link"/>
         <child link="lidar_link"/>
@@ -15,5 +17,5 @@
         </visual>
         <collision>
-            <origin  xyz="0 0 ${link1_height/2}" rpy="0 0 0"/>
+            <origin  xyz="0 0 0" rpy="0 0 0"/>
             <geometry>
                 <cylinder radius= "0.03" length="0.08"/>
