Commit message: teleop ready for arm

File: control_ws/src/lotti_control/description/ros2_control/Lotti.ros_control.xacro (robot description, xacro)
@@ -9,8 +9,4 @@
         </hardware>
         <joint name="arm_link1_joint">
-            <command_interface name="position">
-                <!-- <param name="min">${-pi/2}</param> -->
-                <!-- <param name="max">${pi/2}</param> -->
-            </command_interface>
             <command_interface name="velocity"/>
             <state_interface name="position"/>
@@ -20,8 +16,4 @@
         </joint>
         <joint name="arm_link2_joint">
-            <command_interface name="position">
-                <!-- <param name="min">${-pi/2}</param> -->
-                <!-- <param name="max">${pi/2}</param> -->
-            </command_interface>
             <command_interface name="velocity"/>
             <state_interface name="position"/>
@@ -31,8 +23,4 @@
         </joint>
         <joint name="arm_link3_joint">
-            <command_interface name="position">
-                <!-- <param name="min">${-pi/2}</param> -->
-                <!-- <param name="max">${pi/2}</param> -->
-            </command_interface>
             <command_interface name="velocity"/>
             <state_interface name="position"/>
@@ -42,8 +30,4 @@
         </joint>
         <joint name="arm_link4_joint">
-            <command_interface name="position">
-                <!-- <param name="min">${-pi/2}</param> -->
-                <!-- <param name="max">${pi/2}</param> -->
-            </command_interface>
             <command_interface name="velocity"/>
             <state_interface name="position"/>
@@ -53,8 +37,4 @@
         </joint>
         <joint name="arm_link5_joint">
-            <command_interface name="position">
-                <!-- <param name="min">${-pi/3}</param> -->
-                <!-- <param name="max">${pi/3}</param> -->
-            </command_interface>
             <command_interface name="velocity"/>
             <state_interface name="position"/>
@@ -64,8 +44,4 @@
         </joint>
         <joint name="arm_link6_joint">
-            <command_interface name="position">
-                <!-- <param name="min">${-pi}</param> -->
-                <!-- <param name="max">${pi}</param> -->
-            </command_interface>
             <command_interface name="velocity"/>
             <state_interface name="position"/>

File: control_ws/src/lotti_control/description/urdf/Lotti_body.xacro (robot description, xacro)
@@ -15,8 +15,9 @@
         </visual>
         <collision>
-            <!-- <origin rpy="0 0 0" xyz="0 0 ${(body_height/2)}"/>
+            <origin rpy="0 0 0" xyz="0 0 ${(body_height/2)}"/>
             <geometry>
-                <box size="${body_length} ${body_width} ${body_height}"/>
-            </geometry> -->
+                <box size="0.1 0.1 0.1"/>
+                <!-- <box size="${body_length} ${body_width} ${body_height}"/> -->
+            </geometry>
         </collision>
         <innertial></innertial>

Commit message: flipper working

File: control_ws/src/lotti_control/description/ros2_control/Lotti.ros_control.xacro (robot description, xacro)
@@ -77,5 +77,4 @@
             <param name="left_wheel_name">left_chain_joint</param>
             <param name="right_wheel_name">right_chain_joint</param>
-            <param name="enc_counts_per_rev">3436</param>
         </hardware>
         <joint name="left_chain_joint">

File: control_ws/src/lotti_control/description/urdf/Lotti.urdf.xacro (robot description, xacro)
@@ -11,4 +11,4 @@
     <xacro:include filename="$(find lotti_control)/ros2_control/Lotti.ros_control.xacro"/>
 <!-- world origin -->
-    <link name="world"></link>
+    <!-- <link name="world"></link> -->
 </robot>

File: control_ws/src/lotti_control/description/urdf/Lotti_body.xacro (robot description, xacro)
@@ -6,10 +6,10 @@
     <xacro:property name="body_height" value="0.15"/>
     <xacro:property name="body_mass" value="25.0"/>
-    <joint name="world_joint" type="fixed">
+<!--     <joint name="world_joint" type="floating">
         <origin xyz="0 0 0" rpy="0 0 0"/>
         <parent link="world"/>
         <child link="body_link"/>
         <axis xyz="0 0 0"/>
-    </joint>
+    </joint>  -->
     <link name="body_link">
         <visual>

Commit message: ready for Pi

File: control_ws/src/lotti_control/description/ros2_control/Lotti.ros_control.xacro (robot description, xacro)
@@ -1,10 +1,14 @@
 <?xml version="1.0"?>
 <robot xmlns:xacro="http://www.ros.org/wiki/xacro" >
+    <!-- Arduino device IDs:
+    1: /dev/serial/by-id/usb-Arduino__www.arduino.cc__0043_8503331313735151A0F0-if00
+    2:
+    3:
+    4:
+     -->
     <ros2_control name="LottiArm" type="system">
         <hardware>
             <plugin>arm_interface/ArmInterface</plugin>
-            <!-- <param name="arm_enc_res">4096</param> -->
-            <!-- <param name="arm_max_torque">${9.81*30/100}</param> -->
-            <!-- <param name="arm_max_volt">12</param>           -->
+            <param name="device">/dev/serial/by-id/</param>
         </hardware>
         <joint name="arm_link1_joint">
@@ -54,4 +58,5 @@
         <hardware>
             <plugin>flipper_interface/FlipperInterface</plugin>
+            <param name="device">/dev/serial/by-id/usb-Arduino__www.arduino.cc__0043_8503331313735151A0F0-if00</param>
         </hardware>
         <joint name="flipper_fr_joint">
@@ -89,28 +94,3 @@
         </joint>
     </ros2_control>
-<!--
-        <ros2_control name="LottiChains" type="system">
-        <hardware>
-            <plugin>chain_interface/ChainInterface</plugin>
-            <param name="chains_max_speed" value="28"/>
-            <param name="chains_max_torque" value="20"/>
-        </hardware>
-        <joint name="left_chain_joint">
-            <command_interface name="velocity"/>
-            <command_interface name="torque"/>
-            <state_interface name="position"/>
-            <state_interface name="velocity"/>
-            <state_interface name="torque"/>
-            <state_interface name="temp"/>
-        </joint>
-        <joint name="right_chain_joint">
-            <command_interface name="velocity"/>
-            <command_interface name="torque"/>
-            <state_interface name="position"/>
-            <state_interface name="velocity"/>
-            <state_interface name="torque"/>
-            <state_interface name="temp"/>
-        </joint>
-    </ros2_control>
- -->
 </robot>

Commit message: working arm

File: control_ws/src/lotti_control/description/ros2_control/Lotti.ros_control.xacro (robot description, xacro)
@@ -9,9 +9,10 @@
     Mega1 usb-Arduino__www.arduino.cc__0042_950353139353515082C1-if00
     Mega2 usb-Arduino__www.arduino.cc__0042_8513030353835180A0B1-if00
+    usb-Arduino_LLC_Arduino_Leonardo-if00
     -->
     <ros2_control name="LottiArm" type="system" rw_rate="20">
         <hardware>
             <plugin>arm_interface/ArmInterface</plugin>
-            <param name="device">/dev/serial/by-id/usb-Arduino__www.arduino.cc__0042_950353139353515082C1-if00</param>
+            <param name="device">/dev/serial/by-id/usb-Arduino_LLC_Arduino_Leonardo-if00</param>
             <param name="maxSpeed">2000</param>
         </hardware>
@@ -112,3 +113,20 @@
         </joint>
     </ros2_control>
+    <!-- <ros2_control name="LottiChains" type="system">
+        <hardware>
+            <plugin>diffdrive_lotti/DiffDriveLotti</plugin>
+            <param name="left_wheel_name">left_chain_joint</param>
+            <param name="right_wheel_name">right_chain_joint</param>
+        </hardware>
+        <joint name="left_chain_joint">
+            <command_interface name="velocity"/>
+            <state_interface name="position"/>
+            <state_interface name="velocity"/>
+        </joint>
+        <joint name="right_chain_joint">
+            <command_interface name="velocity"/>
+            <state_interface name="position"/>
+            <state_interface name="velocity"/>
+        </joint>
+    </ros2_control> -->
 </robot>

File: control_ws/src/lotti_control/description/urdf/Lotti_arm.xacro (robot description, xacro)
@@ -57,13 +57,13 @@
   </link>
   <joint name="arm_link1_joint" type="revolute">
-    <origin xyz="0 0 0.0813" rpy="0 0 1.5708" />
+    <origin xyz="0 0 0.0813" rpy="0 0 3.1416" />
     <parent link="arm_base_link" />
     <child link="arm_link1_link" />
     <axis xyz="0 0 -1" />
     <limit
-      lower="-3"
-      upper="3"
-      effort="3"
-      velocity="0.5" />
+      lower="0"
+      upper="3.2"
+      effort="3"
+      velocity="1" />
   </joint>
   <link name="arm_link2_link">
@@ -199,5 +199,5 @@
       upper="3"
       effort="3"
-      velocity="1" />
+      velocity="2" />
   </joint>
   <link name="arm_link6_link">
