Commit message: Add Gazebo Classic simulation support for Lotti3
- Add Lotti_gazebo_control.xacro with friction properties and gazebo_ros2_control plugin
- Add Lotti_sim.ros2_control.xacro using GazeboSystem instead of serial hardware plugins
- Add lotti_world.world (flat ground + sun SDF world)
- Add gazebo.launch.py: full sim stack (Gazebo → spawn → controllers → MoveIt/Servo → teleop → RViz)
- Add use_sim xacro arg to Lotti.urdf.xacro with conditional hardware branching
- Fix chain joints fixed→continuous in Lotti_body.xacro; fix empty body inertia
- Add description/worlds to CMakeLists.txt install rule
- Add package.xml for lotti_control3 (was missing); includes gazebo_ros2_control deps
- Add CLAUDE.md with project context and simulation usage docs

Real hardware launches (robot.launch.py, full.launch.py) are untouched.
Launch sim: ros2 launch lotti_control3 gazebo.launch.py

Co-Authored-By: Claude Sonnet 4.6 <noreply@anthropic.com>

File: control_ws/src/lotti_control3/description/urdf/Lotti.urdf.xacro (robot description, xacro)
@@ -1,4 +1,6 @@
 <?xml version="1.0"?>
 <robot xmlns:xacro="http://www.ros.org/wiki/xacro" name="Lotti3">
+<!-- Simulation switch: pass use_sim:=true for Gazebo, default is real hardware -->
+    <xacro:arg name="use_sim" default="false"/>
 <!-- included files for properties -->
     <xacro:include filename="urdf_inertial_shapes.xacro" />
@@ -8,7 +10,12 @@
     <xacro:include filename="Lotti_body.xacro"/>
     <!-- <xacro:include filename="Lotti_lidar.xacro"/> -->
-<!-- include controllers -->
-<!-- <xacro:include filename="Lotti_gazebo_control.xacro"/> -->
-    <xacro:include filename="$(find lotti_control3)/ros2_control/Lotti.ros2_control.xacro"/>
+<!-- include controllers — switches between simulation and real hardware plugins -->
+    <xacro:if value="$(arg use_sim)">
+        <xacro:include filename="Lotti_gazebo_control.xacro"/>
+        <xacro:include filename="$(find lotti_control3)/ros2_control/Lotti_sim.ros2_control.xacro"/>
+    </xacro:if>
+    <xacro:unless value="$(arg use_sim)">
+        <xacro:include filename="$(find lotti_control3)/ros2_control/Lotti.ros2_control.xacro"/>
+    </xacro:unless>
 <!-- world origin -->
 <!--     <link name="world"></link> -->

File: control_ws/src/lotti_control3/description/urdf/Lotti_body.xacro (robot description, xacro)
@@ -22,12 +22,10 @@
             <origin rpy="0 0 0" xyz="0 0 ${(body_height/2)}"/>
             <geometry>
-                <box size="0.1 0.1 0.1"/>
-                <!-- <box size="${body_length} ${body_width} ${body_height}"/> -->
+                <box size="${body_length} ${body_width} ${body_height}"/>
             </geometry>
         </collision>
-        <innertial></innertial>
-        <!-- <xacro:inertial_box mass="${body_mass}" x="${body_length}" y="${body_width}" z="${body_height}">
+        <xacro:inertial_box mass="${body_mass}" x="${body_length}" y="${body_width}" z="${body_height}">
             <origin rpy="0 0 0" xyz="0 0 ${(body_height/2)}"/>
-        </xacro:inertial_box> -->
+        </xacro:inertial_box>
     </link>
 <!-- Chains (represented by wheels) -->
@@ -59,5 +57,5 @@
 <!-- Left Chain-->
 <!-- Main Wheel-->
-    <joint name="left_chain_joint" type="fixed">
+    <joint name="left_chain_joint" type="continuous">
         <origin xyz="0 ${wheel_seperation/2} ${wheel_radius}" rpy="0 0 0"/>
         <parent link="body_link"/>
@@ -68,5 +66,5 @@
 <!-- Right Chain-->
 <!-- Main Wheel-->
-    <joint name="right_chain_joint" type="fixed">
+    <joint name="right_chain_joint" type="continuous">
         <origin xyz="0 ${-wheel_seperation/2} ${wheel_radius}" rpy="0 0 0"/>
         <parent link="body_link"/>
