Commit message: CubeMars working

File: src/lotti2_control/description/urdf/Lotti_body.xacro (robot description, xacro)
@@ -84,5 +84,5 @@
         <parent link="body_link"/>
         <child link="left_chain_link"/>
-        <axis xyz="0 1 0"/>
+        <axis xyz="0 -1 0"/>
     </joint>
     <xacro:chain_link position="left"/>
