Commit message: reworked flipper control.

File: src/lotti2_control/description/ros2_control/Lotti2.ros2_control.xacro (robot description, xacro)
@@ -4,12 +4,10 @@
         <hardware>
             <plugin>lotti2_flipper_interface/FlipperInterface</plugin>
-            <param name="device_1"></param>
-            <param name="device_2"></param>
-            <param name="positional_stiffness">0.95</param>
+            <param name="device">/dev/serial/by-id/usb-FTDI_USB__-__Serial_Converter_FTAD5NYU-if00-port0</param>
+            <param name="max_torque">0.006</param>
             <param name="gear_ratio">1.0</param>
-            <param name="use_hardware">0</param>
+            <param name="use_hardware">1</param>
         </hardware>
         <joint name="flipper_fr_joint">
-            <command_interface name="position"/>
             <command_interface name="effort"/>
             <state_interface name="position"/>
@@ -19,5 +17,4 @@
         </joint>
         <joint name="flipper_fl_joint">
-            <command_interface name="position"/>
             <command_interface name="effort"/>
             <state_interface name="position"/>
@@ -27,5 +24,4 @@
         </joint>
         <joint name="flipper_rr_joint">
-            <command_interface name="position"/>
             <command_interface name="effort"/>
             <state_interface name="position"/>
@@ -35,5 +31,4 @@
         </joint>
         <joint name="flipper_rl_joint">
-            <command_interface name="position"/>
             <command_interface name="effort"/>
             <state_interface name="position"/>
@@ -54,5 +49,5 @@
         <joint name="left_chain_joint">
             <command_interface name="velocity"/>
-            <state_interface name"position"/>
+            <state_interface name="position"/>
             <state_interface name="velocity"/>
             <state_interface name="effort"/>
@@ -61,5 +56,5 @@
         <joint name="right_chain_joint">
             <command_interface name="velocity"/>
-            <state_interface name"position"/>
+            <state_interface name="position"/>
             <state_interface name="velocity"/>
             <state_interface name="effort"/>
@@ -67,49 +62,3 @@
         </joint>
     </ros2_control>
-    <ros2_control name="Lotti2Arm" type="system" rw_rate="50">
-        <hardware>
-            <plugin>lotti2_arm_interface/ArmInterface</plugin>
-            <param name="device"></param>               <!-- name of serial device used to sommunicate with the motors -->
-            <param name="use_synchronization">0</param> <!-- motors can be forced to execute commands synchronously -->
-            <param name="gear_ratio">40.0</param>        <!-- gear ration of cycloidal gears in arm assembly -->
-            <param name="resolution">16384</param>      <!-- steps per one full motor rotation-->
-            <param name="acceleration">2</param>         <!-- motor acceleration | max 255-->
-            <param name="use_hardware">0</param>        <!-- set to 1 of physical hardware is used. Set to 0 if only digital representation is used -->
-        </hardware>
-        <joint name="arm_link1_joint">
-            <command_interface name="position"/>
-            <command_interface name="velocity"/>
-            <state_interface name="position"/>
-            <state_interface name="velocity"/>
-        </joint>
-        <joint name="arm_link2_joint">
-            <command_interface name="position"/>
-            <command_interface name="velocity"/>
-            <state_interface name="position"/>
-            <state_interface name="velocity"/>
-        </joint>
-        <joint name="arm_link3_joint">
-            <command_interface name="position"/>
-            <command_interface name="velocity"/>
-            <state_interface name="position"/>
-            <state_interface name="velocity"/>
-        </joint>
-        <joint name="arm_link4_joint">
-            <command_interface name="position"/>
-            <command_interface name="velocity"/>
-            <state_interface name="position"/>
-            <state_interface name="velocity"/>
-        </joint>
-        <joint name="arm_link5_joint">
-            <command_interface name="position"/>
-            <command_interface name="velocity"/>
-            <state_interface name="position"/>
-            <state_interface name="velocity"/>
-        </joint>
-        <joint name="arm_link6_joint">
-            <command_interface name="position"/>
-            <command_interface name="velocity"/>
-            <state_interface name="position"/>
-            <state_interface name="velocity"/>
-        </joint>
 </robot>

File: src/lotti2_control/description/urdf/Lotti.urdf.xacro (robot description, xacro)
@@ -1,4 +1,4 @@
 <?xml version="1.0"?>
-<robot xmlns:xacro="http://www.ros.org/wiki/xacro" name="Lotti3">
+<robot xmlns:xacro="http://www.ros.org/wiki/xacro" name="Lotti2">
 <!-- included files for properties -->
     <xacro:include filename="urdf_inertial_shapes.xacro" />

Commit message: flipper working in position mode

File: src/lotti2_control/description/ros2_control/Lotti2.ros2_control.xacro (robot description, xacro)
@@ -4,11 +4,11 @@
         <hardware>
             <plugin>lotti2_flipper_interface/FlipperInterface</plugin>
-            <param name="device">/dev/serial/by-id/usb-FTDI_USB__-__Serial_Converter_FTAD5NYU-if00-port0</param>
-            <param name="max_torque">0.006</param>
-            <param name="gear_ratio">1.0</param>
-            <param name="use_hardware">0</param>
+            <param name="device">/dev/serial/by-id/usb-FTDI_USB__-__Serial_Converter_FTA2HIEQ-if00-port0</param>
+           <!--  <param name="max_torque">0.006</param> -->
+            <!-- <param name="gear_ratio">1.0</param> -->
+            <param name="use_hardware">1</param>
         </hardware>
         <joint name="flipper_fr_joint">
-            <command_interface name="effort"/>
+            <command_interface name="position"/>
             <state_interface name="position"/>
             <state_interface name="velocity"/>
@@ -17,5 +17,5 @@
         </joint>
         <joint name="flipper_fl_joint">
-            <command_interface name="effort"/>
+            <command_interface name="position"/>
             <state_interface name="position"/>
             <state_interface name="velocity"/>
@@ -24,5 +24,5 @@
         </joint>
         <joint name="flipper_rr_joint">
-            <command_interface name="effort"/>
+            <command_interface name="position"/>
             <state_interface name="position"/>
             <state_interface name="velocity"/>
@@ -31,5 +31,5 @@
         </joint>
         <joint name="flipper_rl_joint">
-            <command_interface name="effort"/>
+            <command_interface name="position"/>
             <state_interface name="position"/>
             <state_interface name="velocity"/>
@@ -45,5 +45,5 @@
             <param name="gear_ratio">9</param>      <!-- gearbox ratio -->
             <param name="Kt">0.198</param>          <!-- Kt value for the motor [Nm/A] -->
-            <param name="use_hardware">1</param>
+            <param name="use_hardware">0</param>
         </hardware>
         <joint name="left_chain_joint">

File: src/lotti2_control/description/urdf/Lotti_body.xacro (robot description, xacro)
@@ -57,26 +57,4 @@
         </link>
     </xacro:macro>
-<!--
-    <xacro:macro name="chain_link" params="position">
-        <link name="${position}_chain_link">
-            <visual>
-                <origin xyz="0 0 0" rpy="${pi/2} 0 0"/>
-                <geometry>
-                    <cylinder length="${wheel_length}" radius="${wheel_radius}"/>
-                </geometry>
-                <material name="white"/>
-            </visual>
-            <collision>
-                <origin xyz="0 0 0" rpy="${pi/2} 0 0"/>
-                <geometry>
-                    <cylinder length="${wheel_length}" radius="${wheel_radius}"/>
-                </geometry>
-            </collision>
-            <xacro:inertial_cylinder mass="${wheel_mass}" length="${wheel_length}" radius="${wheel_radius}">
-                <origin xyz="0 0 0" rpy="${pi/2} 0 0"/>
-            </xacro:inertial_cylinder>
-        </link>
-    </xacro:macro>
--->
     <!-- Left Chain-->
     <joint name="left_chain_joint" type="continuous">
